File: PCB/is0Topre.kicad_sch (KiCad schematic)
At the start: 29 parts, among them Q1 2N7002, SW1 SW_Push, SW2 EC_SW, U1 ATmega32U4-M, U2 OPA350, Y1 16MHz

Commit message: Fix for resistor missing
Parts:
- added R12: 100k, Resistor_SMD:R_0603_1608Metric, symbol Device:R
Connections:
- net GND: now also R12.1
- net ROW0: now also R12.2
Changed lines of the file:
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@@
   (junction (at 178.435 57.785) (diameter 0) (color 0 0 0 0)
+  )
+  (junction (at 119.38 34.925) (diameter 0) (color 0 0 0 0)
   )
   (junction (at 39.37 54.61) (diameter 0) (color 0 0 0 0)
@@
     (stroke (width 0) (type default) (color 0 0 0 0))
   )
-  (polyline (pts (xy 128.27 12.7) (xy 128.27 53.975))
-    (stroke (width 0) (type default) (color 0 0 0 0))
-  )
-  (polyline (pts (xy 128.27 12.7) (xy 264.16 12.7))
+  (polyline (pts (xy 132.715 12.7) (xy 132.715 53.975))
+    (stroke (width 0) (type default) (color 0 0 0 0))
+  )
+  (polyline (pts (xy 132.715 12.7) (xy 264.16 12.7))
     (stroke (width 0) (type default) (color 0 0 0 0))
   )
@@
     (stroke (width 0) (type default) (color 0 0 0 0))
   )
-  (wire (pts (xy 116.205 34.925) (xy 118.745 34.925))
+  (wire (pts (xy 116.205 34.925) (xy 119.38 34.925))
     (stroke (width 0) (type default) (color 0 0 0 0))
   )
@@
     (stroke (width 0) (type default) (color 0 0 0 0))
   )
+  (wire (pts (xy 119.38 34.925) (xy 119.38 36.83))
+    (stroke (width 0) (type default) (color 0 0 0 0))
+  )
   (wire (pts (xy 50.8 46.99) (xy 56.515 46.99))
     (stroke (width 0) (type default) (color 0 0 0 0))
@@
     (stroke (width 0) (type default) (color 0 0 0 0))
   )
+  (wire (pts (xy 119.38 34.925) (xy 123.825 34.925))
+    (stroke (width 0) (type default) (color 0 0 0 0))
+  )
   (wire (pts (xy 245.11 43.815) (xy 247.65 43.815))
     (stroke (width 0) (type default) (color 0 0 0 0))
@@
     (stroke (width 0) (type default) (color 0 0 0 0))
   )
-  (polyline (pts (xy 89.535 12.7) (xy 128.27 12.7))
+  (polyline (pts (xy 89.535 12.7) (xy 132.715 12.7))
     (stroke (width 0) (type default) (color 0 0 0 0))
   )
@@
     (effects (font (size 1.27 1.27)) (justify left bottom))
   )
-  (text "Analog Gain" (at 129.54 15.24 0)
+  (text "Analog Gain" (at 133.35 15.24 0)
     (effects (font (size 1.27 1.27)) (justify left bottom))
   )
@@
     )
   )
-  (global_label "ROW0" (shape output) (at 118.745 34.925 0) (fields_autoplaced)
+  (global_label "ROW0" (shape output) (at 123.825 34.925 0) (fields_autoplaced)
     (effects (font (size 1.27 1.27)) (justify left))
-    (property "Intersheet References" "${INTERSHEET_REFS}" (id 0) (at 126.4195 34.8456 0)
+    (property "Intersheet References" "${INTERSHEET_REFS}" (id 0) (at 131.4995 34.8456 0)
       (effects (font (size 1.27 1.27)) (justify left) hide)
     )
@@
     (pin "1")
   )
+  (symbol (lib_id "power:GND") (at 119.38 44.45 0) (unit 1)
+    (in_bom yes) (on_board yes) (fields_autoplaced)
+    (property "Reference" "#PWR027" (id 0) (at 119.38 50.8 0)
+      (effects (font (size 1.27 1.27)) hide)
+    )
+    (property "Value" "GND" (id 1) (at 119.38 48.8934 0))
+    (property "Footprint" "" (id 2) (at 119.38 44.45 0)
+      (effects (font (size 1.27 1.27)) hide)
+    )
+    (property "Datasheet" "" (id 3) (at 119.38 44.45 0)
+      (effects (font (size 1.27 1.27)) hide)
+    )
+    (pin "1")
+  )
   (symbol (lib_id "power:GND") (at 108.585 42.545 0) (unit 1)
     (in_bom yes) (on_board yes) (fields_autoplaced)
@@
     )
     (pin "1")
+  )
+  (symbol (lib_id "Device:R") (at 119.38 40.64 180) (unit 1)
+    (in_bom yes) (on_board yes) (fields_autoplaced)
+    (property "Reference" "R12" (id 0) (at 121.158 39.7315 0)
+      (effects (font (size 1.27 1.27)) (justify right))
+    )
+    (property "Value" "100k" (id 1) (at 121.158 42.5066 0)
+      (effects (font (size 1.27 1.27)) (justify right))
+    )
+    (property "Footprint" "Resistor_SMD:R_0603_1608Metric" (id 2) (at 121.158 40.64 90)
+      (effects (font (size 1.27 1.27)) hide)
+    )
+    (property "Datasheet" "~" (id 3) (at 119.38 40.64 0)
+      (effects (font (size 1.27 1.27)) hide)
+    )
+    (pin "1")
+    (pin "2")
   )
   (symbol (lib_id "power:GND") (at 151.13 141.605 0) (unit 1)
@@
       (reference "#PWR026") (unit 1) (value "GND") (footprint "")
     )
+    (path "/01e3da0e-81b4-4ad8-a06d-cca81184a0f8"
+      (reference "#PWR027") (unit 1) (value "GND") (footprint "")
+    )
     (path "/394c73d1-22fb-42a4-a01d-4812c0448a98"
       (reference "#PWR028") (unit 1) (value "GND") (footprint "")
@@
       (reference "R11") (unit 1) (value "100") (footprint "Resistor_SMD:R_0603_1608Metric")
     )
+    (path "/091289bb-f08f-4df2-9890-d8e4d5fe0484"
+      (reference "R12") (unit 1) (value "100k") (footprint "Resistor_SMD:R_0603_1608Metric")
+    )
     (path "/8d3913c2-0e55-4ca1-9451-666d34d20b10"

Commit message: Update of circuit after PCB testing
Parts:
- removed Q1: 2N7002, Package_TO_SOT_SMD:SOT-23, symbol Transistor_FET:2N7002
- removed R7: 100, Resistor_SMD:R_0603_1608Metric, symbol Device:R
- removed R8: 100k, Resistor_SMD:R_0603_1608Metric, symbol Device:R
- added D2: SK6812MINI, LED_SMD:LED_SK6812MINI_PLCC4_3.5x3.5mm_P1.75mm, symbol cipulot_parts:SK6812MINI
- R8: renamed from R10; value 47k -> 100k
- renumbered R9 to R7
Connections:
- net ROW0 is gone; now on net DISCHARGE_PIN: C8.1, R12.2, SW2.2, U2.3 (IN+)
- net GND: now also D2.2 (VSS)
- net VCC: now also D2.4 (VDD)
- net LED: now reaches U1.39 (PF4)
- net LED: now also D2.3 (DIN)
Other:
- note added: "LED"

Commit message: Update for 3d models
Parts:
- SW2: footprint cipulot_parts:ecs_pad_no_ring -> cipulot_parts:ecs_pad_2U_no_ring
Changed lines of the file:
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@@
     (property "Reference" "SW2" (id 0) (at 108.585 29.0662 0))
     (property "Value" "EC_SW" (id 1) (at 108.585 31.6031 0))
-    (property "Footprint" "cipulot_parts:ecs_pad_no_ring" (id 2) (at 108.585 34.925 0)
+    (property "Footprint" "cipulot_parts:ecs_pad_2U_no_ring" (id 2) (at 108.585 34.925 0)
       (effects (font (size 1.27 1.27)) hide)
     )
@@
     )
     (path "/a624124f-26d6-4381-9f5a-a6c85c0560d9"
-      (reference "SW2") (unit 1) (value "EC_SW") (footprint "cipulot_parts:ecs_pad_no_ring")
+      (reference "SW2") (unit 1) (value "EC_SW") (footprint "cipulot_parts:ecs_pad_2U_no_ring")
     )
     (path "/9a2e3747-4807-449c-9a6e-97403e63f36c"
